File: Hardware/Electronic/Backplane/Kicad/_autosave-OTB-backplane.sch (KiCad schematic (older format))
At the start: 1 part

Commit message: Choixe uC + start assign
Other:
- note added: "STM32H725ZGT6\nF:3576963 \n\nserie STM32H735 pobablement compatible"
Changed lines of the file:
@@
 F29 "MEM_I2C_SCL" I L 9950 4150 50
 $EndSheet
+Text Notes 1550 2600 0    50   ~ 0
+STM32H725ZGT6\nF:3576963 \n\nserie STM32H735 pobablement compatible
 $EndSCHEMATC
