File: Hardware/Electronic/Backplane/Kicad/OTB-backplane.sch (KiCad schematic (older format))
At the start: 1 part

Commit message: Choixe uC + start assign
Other:
- note added: "STM32H735VGT5\nF:3576961\n\nserie STM32H725 pobablement compatible"
Changed lines of the file:
@@
 F29 "MEM_I2C_SCL" I L 9950 4150 50
 $EndSheet
+Text Notes 1550 2600 0    50   ~ 0
+STM32H735VGT5\nF:3576961\n\nserie STM32H725 pobablement compatible
 $EndSCHEMATC

Commit message: choice uC + assign
Other:
- note added: "STM32H725ZGT6\nF:3576963 \n\nserie STM32H735 pobablement compatible"
- note removed: "STM32H735VGT5\nF:3576961\n\nserie STM32H725 pobablement compatible"
Changed lines of the file:
@@
 $EndSheet
 Text Notes 1550 2600 0    50   ~ 0
-STM32H735VGT5\nF:3576961\n\nserie STM32H725 pobablement compatible
+STM32H725ZGT6\nF:3576963 \n\nserie STM32H735 pobablement compatible
 $EndSCHEMATC

Commit message: stm32h7 symbol made
Parts:
- added U??: STM32H725Z, symbol myLibS:STM32H725Z

Commit message: assign uC OK
Parts:
- U??: symbol myLibS:STM32H725Z -> OTB-backplane-rescue:STM32H725Z-myLibS
Connections:
- net labels added: ETH_CRS_DV, ETH_MDC, ETH_MDIO, ETH_REF_CLK, ETH_RXD0, ETH_RXD1, ETH_TXD0, ETH_TXD1, ETH_TX_EN, GPIO_0_0, GPIO_0_1, GPIO_0_2, GPIO_0_3, GPIO_0_4, GPIO_0_5, GPIO_0_6, GPIO_0_7, GPIO_1_0, GPIO_1_1, GPIO_1_2, GPIO_1_3, GPIO_1_4, GPIO_1_5, GPIO_1_6, GPIO_1_7, GPIO_2_0, GPIO_2_1, GPIO_2_2, GPIO_2_3, GPIO_2_4, GPIO_2_5, GPIO_2_6, GPIO_2_7, GPIO_3_0, GPIO_3_1, GPIO_3_2, GPIO_3_3, GPIO_3_4, GPIO_3_5, GPIO_3_6, GPIO_3_7, I2C1_SCL, I2C1_SDA, I2C2_SCL, I2C2_SDA, I2C3_SCL, I2C3_SDA, I2C4_SCL, I2C4_SDA, I2C5_SCL, I2C5_SDA, JTCK_SWCLK, JTMS_SWDIO, SPI1_MISO, SPI1_MOSI, SPI1_NSS, SPI1_SCK, SPI2_MISO, SPI2_MOSI, SPI2_NSS, SPI2_SCK, SPI3_MISO, SPI3_MOSI, SPI3_NSS, SPI3_SCK, SPI4_MISO, SPI4_MOSI, SPI4_NSS, SPI4_SCK, SPI5_MISO, SPI5_MOSI, SPI5_NSS, SPI5_SCK, UART4_RTS, UART4_RX, UART4_TX, UART7_CTS, UART7_RTS, UART7_RX, UART7_TX, USAR4_CTS, USART1_CTS, USART1_RTS, USART1_RX, USART1_TX, USART2_CTS, USART2_RTS, USART2_RX, USART2_TX, USART3_CTS, USART3_RTS, USART3_RX, USART3_TX, USART6_CTS, USART6_RTS, USART6_RX, USART6_TX
Other:
- note added: "PC"
- note added: "RCC_osc"

Commit message: Switch stm32h725 to stm32h723
Parts:
- added U?: STM32H723ZG, Package_QFP:LQFP-144_20x20mm_P0.5mm, symbol MCU_ST_STM32H7:STM32H743ZITx
Other:
- moved on the sheet: U??
Changed lines of the file:
@@
 L OTB-backplane-rescue:STM32H725Z-myLibS U??
 U 1 1 60B11ED4
-P 6475 5500
-F 0 "U??" H 6400 1536 150 0000 C CNB
-F 1 "STM32H725Z" H 6400 1295 150 0000 C CNB
-F 2 "" H 275 6100 50  0001 C CNN
-F 3 "" H 275 6100 50  0001 C CNN
-	1    6475 5500
+P -8100 -1925
+F 0 "U??" H -8175 -5889 150 0000 C CNB
+F 1 "STM32H725Z" H -8175 -6130 150 0000 C CNB
+F 2 "" H -14300 -1325 50  0001 C CNN
+F 3 "" H -14300 -1325 50  0001 C CNN
+	1    -8100 -1925
 	1    0    0    -1
 $EndComp
-Text Label 4200 5150 0    50   ~ 0
+Text Label 4850 8000 0    50   ~ 0
 SPI4_NSS
-Text Label 4200 4950 0    50   ~ 0
+Text Label 4850 7800 0    50   ~ 0
 SPI4_SCK
-Text Label 4200 5250 0    50   ~ 0
+Text Label 4850 8100 0    50   ~ 0
 SPI4_MISO
-Text Label 4200 5350 0    50   ~ 0
+Text Label 4850 8200 0    50   ~ 0
 SPI4_MOSI
-Text Label 8600 8250 2    50   ~ 0
+Text Label 4850 6500 0    50   ~ 0
 SPI5_NSS
-Text Label 8600 8350 2    50   ~ 0
+Text Label 4850 6600 0    50   ~ 0
 SPI5_SCK
-Text Label 8600 8450 2    50   ~ 0
+Text Label 4850 6700 0    50   ~ 0
 SPI5_MISO
-Text Label 8600 8550 2    50   ~ 0
+Text Label 4850 7100 0    50   ~ 0
 SPI5_MOSI
-Text Notes 4350 7600 0    50   ~ 0
+Text Notes -10225 175  0    50   ~ 0
 RCC_osc
-Text Label 8600 6800 2    50   ~ 0
+Text Label 8300 6200 2    50   ~ 0
 SPI2_MOSI
-Text Label 8600 6700 2    50   ~ 0
+Text Label 8300 6100 2    50   ~ 0
 SPI2_MISO
-Text Label 8650 3000 2    50   ~ 0
+Text Label 8400 2500 2    50   ~ 0
 USART2_CTS
-Text Label 4125 3400 0    50   ~ 0
+Text Label 8350 8000 2    50   ~ 0
 USART2_RTS
-Text Label 4125 3500 0    50   ~ 0
+Text Label 8350 8100 2    50   ~ 0
 USART2_TX
-Text Label 8650 3300 2    50   ~ 0
+Text Label 8400 2800 2    50   ~ 0
 USART2_RX
 Wire Notes Line
-	8650 3850 8750 3850
-Wire Notes Line
-	8750 3850 8750 4250
-Wire Notes Line
-	8750 4250 8650 4250
-Wire Notes Line
-	8750 4050 8900 4050
-Wire Notes Line
-	8900 4050 8850 4000
-Wire Notes Line
-	8900 4050 8850 4100
-Text Notes 8900 4050 0    50   ~ 0
+	8400 3325 8500 3325
+Wire Notes Line
+	8500 3325 8500 3725
+Wire Notes Line
+	8500 3725 8400 3725
+Wire Notes Line
+	8500 3525 8650 3525
+Wire Notes Line
+	8650 3525 8600 3475
+Wire Notes Line
+	8650 3525 8600 3575
+Text Notes 8650 3525 0    50   ~ 0
 PC
-Text Label 8650 3400 2    50   ~ 0
+Text Label 8400 2900 2    50   ~ 0
 SPI3_NSS
-Text Label 8650 3500 2    50   ~ 0
+Text Label 8400 3000 2    50   ~ 0
 SPI1_SCK
-Text Label 8650 3600 2    50   ~ 0
+Text Label 8400 3100 2    50   ~ 0
 SPI1_MISO
-Text Label 4150 3700 0    50   ~ 0
+Text Label 8350 8300 2    50   ~ 0
 SPI1_MOSI
-Text Label 8700 4750 2    50   ~ 0
+Text Label 8400 4200 2    50   ~ 0
 USAR4_CTS
-Text Label 8700 4950 2    50   ~ 0
+Text Label 8400 4400 2    50   ~ 0
 SPI3_MOSI
-Text Label 8600 8850 2    50   ~ 0
+Text Label 4850 7300 0    50   ~ 0
 I2C4_SCL
-Text Label 8600 8950 2    50   ~ 0
+Text Label 4850 7400 0    50   ~ 0
 I2C4_SDA
-Text Label 4200 5450 0    50   ~ 0
+Text Label 4850 8300 0    50   ~ 0
 UART7_RX
-Text Label 4200 5550 0    50   ~ 0
+Text Label 4850 8400 0    50   ~ 0
 UART7_TX
-Text Label 4150 5650 0    50   ~ 0
+Text Label 4850 8500 0    50   ~ 0
 UART7_RTS
-Text Label 4150 5750 0    50   ~ 0
+Text Label 4850 6800 0    50   ~ 0
 UART7_CTS
-Text Label 8600 5750 2    50   ~ 0
+Text Label 8450 5200 2    50   ~ 0
 I2C2_SCL
-Text Label 8600 5850 2    50   ~ 0
+Text Label 8450 5300 2    50   ~ 0
 I2C2_SDA
-Text Label 8600 5650 2    50   ~ 0
+Text Label 8400 4600 2    50   ~ 0
 SPI2_NSS
-Text Label 8600 6050 2    50   ~ 0
+Text Label 8350 7900 2    50   ~ 0
 SPI2_SCK
-Text Label 8600 6150 2    50   ~ 0
+Text Label 8450 5600 2    50   ~ 0
 UART4_RTS
-Text Label 4150 3800 0    50   ~ 0
+Text Label 8350 8400 2    50   ~ 0
 USART3_TX
-Text Label 4150 3900 0    50   ~ 0
+Text Label 8350 8500 2    50   ~ 0
 USART3_RX
-Text Label 4150 4100 0    50   ~ 0
+Text Label 8450 5500 2    50   ~ 0
 USART3_CTS
-Text Label 4150 4200 0    50   ~ 0
+Text Label 8350 8800 2    50   ~ 0
 USART3_RTS
-Text Label 4100 6700 0    50   ~ 0
+Text Label 4850 5000 0    50   ~ 0
 USART6_RTS
-Text Label 8650 7100 2    50   ~ 0
+Text Label 8300 6500 2    50   ~ 0
 USART6_TX
-Text Label 8650 7200 2    50   ~ 0
+Text Label 8300 6600 2    50   ~ 0
 USART6_RX
-Text Label 8650 7400 2    50   ~ 0
+Text Label 8300 6800 2    50   ~ 0
 I2C3_SDA
-Text Label 8650 3800 2    50   ~ 0
+Text Label 8400 3300 2    50   ~ 0
 I2C3_SCL
-Text Label 8650 3900 2    50   ~ 0
+Text Label 8400 3375 2    50   ~ 0
 USART1_TX
-Text Label 8650 4100 2    50   ~ 0
+Text Label 8400 3575 2    50   ~ 0
 USART1_CTS
-Text Label 8650 4200 2    50   ~ 0
+Text Label 8400 3675 2    50   ~ 0
 USART1_RTS
-Text Label 8650 4300 2    50   ~ 0
+Text Label 8400 3775 2    50   ~ 0
 JTMS_SWDIO
-Text Label 8650 4400 2    50   ~ 0
+Text Label 8400 3875 2    50   ~ 0
 JTCK_SWCLK
-Text Label 8650 4500 2    50   ~ 0
+Text Label 8400 3975 2    50   ~ 0
 SPI1_NSS
-Text Label 8650 7500 2    50   ~ 0
+Text Label 4850 5900 0    50   ~ 0
 I2C5_SDA
-Text Label 8650 7600 2    50   ~ 0
+Text Label 4850 6000 0    50   ~ 0
 I2C5_SCL
-Text Label 4150 3000 0    50   ~ 0
+Text Label 8350 7600 2    50   ~ 0
 UART4_RX
-Text Label 4150 3100 0    50   ~ 0
+Text Label 8350 7700 2    50   ~ 0
 UART4_TX
-Text Label 4100 7200 0    50   ~ 0
+Text Label 4850 5500 0    50   ~ 0
 USART6_CTS
-Text Label 8700 5050 2    50   ~ 0
+Text Label 8300 6900 2    50   ~ 0
 SPI3_SCK
-Text Label 8700 5150 2    50   ~ 0
+Text Label 8300 7000 2    50   ~ 0
 SPI3_MISO
-Text Label 8700 5350 2    50   ~ 0
+Text Label 8400 4800 2    50   ~ 0
 I2C1_SCL
-Text Label 8700 5450 2    50   ~ 0
+Text Label 8400 4900 2    50   ~ 0
 I2C1_SDA
-Text Label 8650 4000 2    50   ~ 0
+Text Label 8400 3475 2    50   ~ 0
 USART1_RX
 Text Label 12000 2625 0    50   ~ 0
@@
 Text Label 13950 7450 0    50   ~ 0
 GPIO_3_7
-Text Label 8600 6600 2    50   ~ 0
+Text Label 8300 6000 2    50   ~ 0
 ETH_MDC
-Text Label 8675 3100 2    50   ~ 0
+Text Label 8400 2600 2    50   ~ 0
 ETH_REF_CLK
-Text Label 8675 3200 2    50   ~ 0
+Text Label 8400 2700 2    50   ~ 0
 ETH_MDIO
-Text Label 8650 3700 2    50   ~ 0
+Text Label 8400 3200 2    50   ~ 0
 ETH_CRS_DV
-Text Label 8600 6900 2    50   ~ 0
+Text Label 8300 6300 2    50   ~ 0
 ETH_RXD0
-Text Label 8600 7000 2    50   ~ 0
+Text Label 8300 6400 2    50   ~ 0
 ETH_RXD1
-Text Label 8600 5950 2    50   ~ 0
+Text Label 8450 5400 2    50   ~ 0
 ETH_TXD0
-Text Label 4100 7000 0    50   ~ 0
+Text Label 4850 5300 0    50   ~ 0
 ETH_TX_EN
-Text Label 4100 7100 0    50   ~ 0
+Text Label 4850 5400 0    50   ~ 0
 ETH_TXD1
-Text Label 4125 3200 0    50   ~ 0
+Text Label 4850 4200 0    50   ~ 0
 GPIO_0_0
-Text Label 4125 3300 0    50   ~ 0
+Text Label 4850 4300 0    50   ~ 0
 GPIO_0_1
-Text Label 4125 3600 0    50   ~ 0
+Text Label 4850 4400 0    50   ~ 0
 GPIO_0_2
-Text Label 4150 4000 0    50   ~ 0
+Text Label 4850 4500 0    50   ~ 0
 GPIO_0_3
-Text Label 4150 4300 0    50   ~ 0
+Text Label 4850 4600 0    50   ~ 0
 GPIO_0_4
-Text Label 4150 4400 0    50   ~ 0
+Text Label 4850 4700 0    50   ~ 0
 GPIO_0_5
-Text Label 4150 4500 0    50   ~ 0
+Text Label 4850 4800 0    50   ~ 0
 GPIO_0_6
-Text Label 4175 4750 0    50   ~ 0
+Text Label 4850 4900 0    50   ~ 0
 GPIO_0_7
-Text Label 4100 6600 0    50   ~ 0
+Text Label 4850 6900 0    50   ~ 0
 GPIO_2_0
-Text Label 4100 6800 0    50   ~ 0
+Text Label 4850 7000 0    50   ~ 0
 GPIO_2_1
-Text Label 4100 6900 0    50   ~ 0
+Text Label 4850 7200 0    50   ~ 0
 GPIO_2_2
-Text Label 4100 7300 0    50   ~ 0
+Text Label 4850 7600 0    50   ~ 0
 GPIO_2_3
-Text Label 8700 4850 2    50   ~ 0
+Text Label 4850 7700 0    50   ~ 0
 GPIO_2_4
-Text Label 8700 5250 2    50   ~ 0
+Text Label 4850 7900 0    50   ~ 0
 GPIO_2_5
-Text Label 8700 5550 2    50   ~ 0
+Text Label 4850 8600 0    50   ~ 0
 GPIO_2_6
-Text Label 8600 6250 2    50   ~ 0
+Text Label 4850 8700 0    50   ~ 0
 GPIO_2_7
-Text Label 4175 4850 0    50   ~ 0
+Text Label 4850 5100 0    50   ~ 0
 GPIO_1_0
-Text Label 4200 5050 0    50   ~ 0
+Text Label 4850 5200 0    50   ~ 0
 GPIO_1_1
-Text Label 4175 5850 0    50   ~ 0
+Text Label 4850 5600 0    50   ~ 0
 GPIO_1_2
-Text Label 4175 5950 0    50   ~ 0
+Text Label 4850 5700 0    50   ~ 0
 GPIO_1_3
-Text Label 4175 6050 0    50   ~ 0
+Text Label 4850 6100 0    50   ~ 0
 GPIO_1_4
-Text Label 4175 6150 0    50   ~ 0
+Text Label 4850 6200 0    50   ~ 0
 GPIO_1_5
-Text Label 4175 6250 0    50   ~ 0
+Text Label 4850 6300 0    50   ~ 0
 GPIO_1_6
-Text Label 4100 6500 0    50   ~ 0
+Text Label 4850 6400 0    50   ~ 0
 GPIO_1_7
-Text Label 8600 6500 2    50   ~ 0
+Text Label 4850 8800 0    50   ~ 0
 GPIO_3_0
-Text Label 8650 7300 2    50   ~ 0
+Text Label 4850 8900 0    50   ~ 0
 GPIO_3_1
-Text Label 8650 7700 2    50   ~ 0
+Text Label 4850 9000 0    50   ~ 0
 GPIO_3_2
-Text Label 8650 7800 2    50   ~ 0
+Text Label 4850 9100 0    50   ~ 0
 GPIO_3_3
-Text Label 8650 7900 2    50   ~ 0
+Text Label 8350 7800 2    50   ~ 0
 GPIO_3_4
-Text Label 8650 8000 2    50   ~ 0
+Text Label 8350 8200 2    50   ~ 0
 GPIO_3_5
-Text Label 8600 8650 2    50   ~ 0
+Text Label 8350 8600 2    50   ~ 0
 GPIO_3_6
-Text Label 8600 8750 2    50   ~ 0
+Text Label 8350 8700 2    50   ~ 0
 GPIO_3_7
+$Comp
+L MCU_ST_STM32H7:STM32H743ZITx U?
+U 1 1 60B5F8A7
+P 6650 5800
+F 0 "U?" H 6600 2111 50  0000 C CNN
+F 1 "STM32H723ZG" H 6600 2020 50  0000 C CNN
+F 2 "Package_QFP:LQFP-144_20x20mm_P0.5mm" H 5550 2400 50  0001 R CNN
+F 3 "http://www.st.com/st-web-ui/static/active/en/resource/technical/document/datasheet/DM00387108.pdf" H 6650 5800 50  0001 C CNN
+	1    6650 5800
+	1    0    0    -1
+$EndComp
 $EndSCHEMATC

Commit message: Update def
Parts:
- removed U??: STM32H725Z, symbol OTB-backplane-rescue:STM32H725Z-myLibS

Commit message: ethernet start
Parts:
- added C?: 100nF, Capacitor_SMD:C_0805_2012Metric, symbol Device:C
- added J?: WR-PHD 2.54 20, symbol Connector_Generic:Conn_02x10_Odd_Even
- added R? (x4): 1K, symbol Device:R
- added R?: 1.5K, symbol Device:R
- added U?: PCA9600D, Package_SO:SO-8_3.9x4.9mm_P1.27mm, symbol Interface:PCA9600D
- added U?: DP83848M, symbol myLibS:DP83848M
- added X?: ASV-50.000MHZ-EJ-T, Oscillator:Oscillator_SMD_Abracon_ASV-4Pin_7.0x5.1mm, symbol Oscillator:ASV-xxxMHz
Connections:
- net +12V: now also J?.1 (Pin_1), J?.2 (Pin_2)
- net ETH_CRS_DV: now also U?.33 (CRS/CRS_DV/LED_CFG)
- net ETH_MDC: now also U?.25 (MDC)
- net ETH_MDIO: now also R?.2, U?.24 (MDIO)
- net ETH_REF_CLK: now also U?.28 (X1), X?.3 (OUT)
- net ETH_RXD0: now also U?.36 (RXD_0/PHYAD1)
- net ETH_RXD1: now also U?.37 (RXD_1/PHYAD2)
- net ETH_TXD0: now also U?.4 (TXD_0)
- net ETH_TXD1: now also U?.5 (TXD_1)
- net ETH_TX_EN: now also U?.3 (TX_EN)
- net GND: now also C?.2, J?.3 (Pin_3), J?.4 (Pin_4), J?.7 (Pin_7), J?.8 (Pin_8), U?.4 (GND), X?.2 (GND)
- net I2C5_SCL: now also R?.2, U?.7 (SY)
- net I2C5_SDA: now also R?.2, U?.1 (SX)
- net SPI5_MISO: now also J?.12 (Pin_12)
- net SPI5_MOSI: now also J?.10 (Pin_10)
- net SPI5_NSS: now also J?.9 (Pin_9)
- net SPI5_SCK: now also J?.11 (Pin_11)
- net UART7_CTS: now also J?.13 (Pin_13)
- net UART7_RTS: now also J?.15 (Pin_15)
- net UART7_RX: now also J?.16 (Pin_16)
- net UART7_TX: now also J?.14 (Pin_14)
- net EN_ETH_CLK: now reaches U?.47 (PB1)
- net EN_ETH_CLK: now also X?.1 (EN)
- new net: J?.17 (Pin_17), R?.2, U?.2 (RX), U?.3 (TX)
- new net: J?.19 (Pin_19), R?.2, U?.5 (TY), U?.6 (RY)
- new net +3V3: C?.1, J?.5 (Pin_5), R?.1, R?.1, R?.1, R?.1, R?.1, X?.4 (Vdd)
- new net +5V: J?.6 (Pin_6)
- no-connect marks 0 -> 6
Other:
- note added: "?"
- note added: "F:3123676"
- moved on the sheet: J?, U?

Commit message: eth on goign
Parts:
- added C? (x7): 100nF, Capacitor_SMD:C_0805_2012Metric, symbol Device:C
- added C?: 10uF 25V, symbol Device:CP
- added J?: Wuerth_7499010121A, Connector_RJ:RJ45_Wuerth_7499010121A_Horizontal, symbol Connector:Wuerth_7499010121A
- added R? (x2): 2K2, symbol Device:R
- added R?: OR, symbol Device:R
- added R? (x3): NM, symbol Device:R
- added R?: 10k, symbol Device:R
- added R?: 4.87K 1%7, symbol Device:R
- added R? (x4): 49.9R, symbol Device:R
- U?: symbol myLibS:DP83848M -> OTB-backplane-rescue:DP83848M-myLibS
Connections:
- net +3V3: now also C?.1, C?.1, C?.1, C?.2, J?.2 (TCT), J?.5 (RCT), R?.1, R?.1, R?.1, R?.1, R?.2, R?.2
- net ETH_CRS_DV: now also R?.1, R?.1; no longer U?.33 (CRS/CRS_DV/LED_CFG)
- net GND: now also C?.1, C?.2, C?.2, C?.2, C?.2, C?.2, C?.2, C?.2, R?.1, R?.1, R?.2, R?.2
- net ~ETH_PHY_RST~: now reaches U?.133 (PB3)
- net ~ETH_PHY_RST~: now also U?.23 (~RESET~), R?.2
- net at U?.11 (RD-): now also J?.6 (RD-), R?.2
- net at U?.12 (RD+): now also J?.4 (RD+), R?.1
- net at U?.14 (TD–): now also J?.3 (TD-), R?.1
- net at U?.15 (TD+): now also J?.1 (TD+), R?.2
- net at U?.16 (PFBIN1): now also U?.19 (PFBOUT), U?.30 (PFBIN2), C?.1, C?.1, C?.1, C?.1
- net at U?.20 (RBIAS): now also R?.2
- net at U?.22 (LED_LINK/AN0): now also R?.2
- net at U?.32 (RX_DV/MII_MODE32): now also R?.2, R?.2
- net at U?.34 (RX_ER/MDIX_EN): now also R?.1
- new net: R?.1, R?.2, U?.33 (CRS/CRS_DV/LED_CFG)
- no-connect marks 6 -> 7
Other:
- note removed: "?"
- moved on the sheet: C?, R?, X?
