File: Hardware/Electronic/Backplane/Kicad/OTB-backplane.sch (KiCad schematic (older format))
At the start: 33 parts

Commit message: ajout ft232h
Parts:
- added C? (x3): 4.7uF, symbol Device:C
- added C? (x10): 100nF, symbol Device:C
- added C? (x2): 4.7uF(NM), symbol Device:C
- added C?: 10nF, symbol Device:C
- added D? (x2): LED, symbol Device:LED
- added FB? (x2): 600R/0.5A, Capacitor_SMD:C_0603_1608Metric, symbol Device:Ferrite_Bead_Small
- added R? (x2): R, symbol Device:R
- added R?: 10K, symbol Device:R
- added R?: 12K, symbol Device:R
- added U?: FT232H, symbol Interface_USB:FT232H
Connections:
- net +3V3: now also C?.1, C?.1, C?.1, C?.1, C?.1, C?.1, C?.1, D?.2 (A), D?.2 (A), FB?.2, FB?.2, R?.2, U?.12 (VCCIO), U?.24 (VCCIO), U?.39 (VCCD), U?.40 (VREGIN), U?.46 (VCCIO)
- net GND: now also C?.2, C?.2, C?.2, C?.2, C?.2, C?.2, C?.2, C?.2, C?.2, C?.2, C?.2, C?.2, C?.2, C?.2, C?.2, C?.2, R?.2, U?.42 (TEST)
- net USART1_CTS: now also U?.15 (ADBUS2)
- net USART1_RTS: now also U?.16 (ADBUS3)
- net USART1_RX: now also U?.13 (ADBUS0)
- net USART1_TX: now also U?.14 (ADBUS1)
- new net: R?.2, U?.27 (ACBUS3)
- new net: R?.2, U?.28 (ACBUS4)
- new net: C?.1, C?.1, FB?.1, U?.3 (VPHY)
- new net: C?.1, R?.1, U?.34 (~RESET)
- new net: C?.1, U?.37 (VCCA)
- new net: C?.1, U?.38 (VCCCORE)
- new net: R?.1, U?.5 (REF)
- new net: C?.1, C?.1, FB?.1, U?.8 (VPLL)
- new net: D?.1 (K), R?.1 (x2)
Other:
- note added: "RX\n"
- note added: "TX\n"
- note added: "VCCD\n"
- note added: "VREGIN"
- moved on the sheet: J?, R?, U?

Commit message: schematic presque ok
Parts:
- added C? (x4): 10uF 25V, Capacitor_SMD:C_0805_2012Metric, symbol Device:C
- added C? (x2): 2.2nF 50V, Capacitor_SMD:C_0402_1005Metric, symbol Device:C
- added C? (x5): 100nF, symbol Device:C
- added C? (x11): 22uF 10V, symbol Device:C
- added C? (x4): 1uF, symbol Device:C
- added C? (x2): 22pF, symbol Device:C
- added C?: 47uF 10V, symbol Device:C
- added C?: 2.2nF, symbol Device:C
- added C?: 3.3nF, symbol Device:C
- added C?: 1nF 1KV, Capacitor_SMD:C_0805_2012Metric, symbol Device:C
- added D? (x3): LED, symbol Device:LED
- added FB? (x2): 8R/10A, Capacitor_SMD:C_0603_1608Metric, symbol Device:Ferrite_Bead_Small
- added FB?: 600R/0.5A, Capacitor_SMD:C_0603_1608Metric, symbol Device:Ferrite_Bead_Small
- added J?: USB_C_Receptacle, symbol Connector:USB_C_Receptacle
- added L? (x2): 2.2uH, symbol Device:L
- added R? (x2): 5K1, symbol Device:R
- added R? (x2): 7.5K 1%, symbol Device:R
- added R?: 2K, symbol Device:R
- added R?: 10K, symbol Device:R
- added R?: 6K8, symbol Device:R
- added R?: 2K15, symbol Device:R
- added R? (x2): 1K, symbol Device:R
- added R?: 6K98, symbol Device:R
- added R?: 1K33, symbol Device:R
- added R?: 470K, symbol Device:R
- added R?: 84K5, symbol Device:R
- added R?: 390K, symbol Device:R
- added R?: 768R, symbol Device:R
- added R?: 47K, symbol Device:R
- added R?: 5K5, symbol Device:R
- added R?: 4.7K, symbol Device:R
- added R?: 275R, symbol Device:R
- added U? (x2): TPS6291x, symbol myLibS:TPS6291x
- added U?: 93LCxxAxxOT, Package_TO_SOT_SMD:SOT-23-6, symbol Memory_EEPROM:93LCxxAxxOT
- added U?: TPS259472x, symbol myLibS:TPS259472x
- added Y?: Crystal, symbol Device:Crystal
- C?: footprint (none) -> Capacitor_SMD:C_0805_2012Metric; PartNo (none) -> C2012X7S1E106K125AC; Supplier (none) -> Mouser: 810-C2012X7S1EK125AC
- J?: PartNo (none) -> 74438356022; Supplier (none) -> Digikey: 732-8232-6-ND
- R?: value NM -> 2K2
Connections:
- net +12V: now also C?.1, C?.1, C?.1, C?.1, C?.1, C?.1, R?.1, R?.2, U?.1 (EN/SYNC), U?.1 (EN/SYNC), U?.6 (OUT), U?.6 (VIN), U?.6 (VIN); no longer J?.1
- net +3V3: now also C?.1, C?.1, U?.8 (VCC), C?.1, C?.1, C?.1, C?.1, C?.2, FB?.1, FB?.1, R?.1, R?.1, R?.2, U?.6 (VCC)
- net +5V: now also C?.1, C?.1, C?.1, C?.1, FB?.1, R?.1, R?.1
- net GND: now also U?.10 (GND), U?.11 (GND), U?.13 (AGND), U?.17 (AGND), U?.22 (GND), U?.23 (GND), U?.29 (DGND), U?.35 (GND), U?.36 (GND), U?.4 (AGND), U?.40 (IOGND), U?.41 (AGND), U?.47 (GND), U?.48 (GND), U?.9 (AGND), C?.1, C?.2, C?.2, C?.2, C?.2, C?.2, C?.2, C?.2, C?.2, C?.2, C?.2, C?.2, C?.2, C?.2, C?.2, C?.2, C?.2, C?.2, C?.2, C?.2, C?.2, C?.2, C?.2, C?.2, C?.2, C?.2, C?.2, C?.2, C?.2, C?.2, D?.1 (K), D?.1 (K), D?.1 (K), J?.A1 (GND), J?.A12 (GND), J?.B1 (GND), J?.B12 (GND), J?.S1 (SHIELD), R?.1, R?.1, R?.2, R?.2, R?.2, R?.2, R?.2, R?.2, R?.2, R?.2, R?.2, U?.2 (GND), U?.4 (PGND), U?.4 (PGND), U?.7 (PSNS), U?.7 (PSNS), U?.8 (GND)
- net LED_LINK: now reaches R?.2, U?.22 (LED_LINK/AN0)
- net LED_LINK: now also J?.10
- net at U?.1 (IOVDD33): now also U?.18 (AVDD33), U?.26 (IOVDD33), C?.1, C?.1, C?.1, C?.1, FB?.2
- net Earth: now reaches J?.8
- net Earth: now also J?.SH, C?.1
- net at J?.9: now also R?.1
- net at U?.1 (XCSI): now also C?.1, Y?.1
- net at U?.2 (XCSO): now also C?.1, Y?.2
- net at U?.43 (EEDATA): now also R?.1, U?.3 (DI)
- net at U?.44 (EECLK): now also U?.4 (CLK)
- net at U?.45 (EECS): now also U?.5 (CS)
- net at U?.6 (DM): now also J?.A7 (D-), J?.B7 (D-)
- net at U?.7 (DP): now also J?.A6 (D+), J?.B6 (D+)
- new net: J?.1, R?.1, U?.5 (IN)
- new net: J?.A5 (CC1), R?.2
- new net: J?.B5 (CC2), R?.2
- new net: R?.1, U?.10 (S-CONF) (x2)
- new net: L?.1, U?.2 (SW) (x2)
- new net: C?.1, C?.1, C?.1, FB?.2, L?.2, U?.3 (VO) (x2)
- new net: C?.1, U?.8 (NR/SS) (x2)
- new net: C?.2, R?.1, R?.2, U?.9 (FB) (x2)
- new net: R?.1, R?.2, U?.1 (DO)
- new net: D?.2 (A), R?.2 (x2)
- new net: R?.1, R?.2, U?.1 (EN/UVLO)
- new net: C?.1, U?.10 (ITIMER)
- new net: R?.1, U?.2 (OVCSEL)
- new net: R?.1, R?.2, U?.3 (PG)
- new net: D?.2 (A), R?.1, U?.4 (PGTH)
- new net: C?.1, U?.7 (dVdt)
- new net: R?.1, U?.9 (ILM)
- new net 5V_USB: J?.A4 (VBUS), J?.A9 (VBUS), J?.B4 (VBUS), J?.B9 (VBUS)
- no-connect marks 7 -> 10
Other:
- note added: "OVC 13.8V\nOVL 8V\nILIM 4A"
- moved on the sheet: C?, D?, FB?, J?, R?, U?, X?
