File: Hardware/Electronic/Backplane/Kicad/periph_conector.sch (KiCad schematic (older format))
At the start: 7 parts

Commit message: Update def
Parts:
- added C?: 100nF, Capacitor_SMD:C_0805_2012Metric, symbol Device:C
- added R?: 10k, symbol Device:R
- added U?: PCA9538, symbol myLibS:PCA9538
Connections:
- net +3V3: now also C?.1, R?.1, U?.16 (VDD)
- net CARD_DETECT_0: now also U?.6 (IO2)
- net CARD_DETECT_1: now also U?.11 (IO6)
- net CTRL_GPIO_0: now also U?.7 (IO3)
- net CTRL_GPIO_1: now also U?.12 (IO7)
- net GND: now also C?.2, U?.8 (VSS)
- net MEM0_SEL: now also U?.4 (IO0)
- net MEM_I2C_SCL: now also U?.14 (SCL)
- net MEM_I2C_SDA: now also U?.15 (SDA)
- net ~MEM_WC_0~: now also U?.5 (IO1)
- net ~MEM_WC_1~: now also U?.10 (IO5)
- net MEM_SEL_1 renamed MEM1_SEL
- net MEM1_SEL: now also U?.9 (IO4)
- new net: R?.2, U?.3 (~RESET)
- new net EXP_A0: U?.1 (A0)
- new net EXP_A1: U?.2 (A1)
Other:
- moved on the sheet: C?, J?
